File: KiCad/ClkController.kicad_sch (KiCad schematic)
At the start: 8 parts, among them SW1 -0.1Mhz, SW2 +0.1Mhz, SW3 -1Mhz, SW4 +1Mhz, U1 ER_OLEDM0.91_1x-I2C, Y1 Si5351A-B-GT, Y2 Modified Oscillator

Commit message: Renamed KiCad Project
Renamed KiCad Project
Other:
- title: Oscillator Controller -> Clk Controller
Changed lines of the file:
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@@
 	(paper "A4")
 	(title_block
-		(title "Oscillator Controller")
+		(title "Clk Controller")
 		(date "2026-08-11")
 		(rev "0.1.0")
